File: labs/LAB 2/K_Circuit_kicad/K_Circuit_kicad.kicad_sch (KiCad schematic)
At the start: 12 parts, among them U1 UA741, U2 UA741, U3 UA741

Commit message: Lab 3 docs
Parts:
- added C1, C2: 4.7u, symbol Device:C
- R3: value 6.8K -> 220k
- R4: value 120K -> 180k
- R5: value 6.8K -> 56k
Connections:
- net at R5.2, R6.1, U2.6: now also C2.2
- net at R4.2, R5.1, U2.3 (+): now also C1.2, C2.1
- net at R3.2, R4.1, U1.6: now also C1.1
Other:
- moved on the sheet: R4
